File: pcb/bancouver40_cfx/bancouver40_cfx.kicad_pcb (KiCad board)
At the start: 2 copper layers, 170 x 69.4 mm, 104 parts, among them J1 USB_C_Receptacle_USB2.0, SW1 SW_Push, SW10 SW_Push, SW11 SW_Push, SW12 SW_Push, SW13 SW_Push, SW14 SW_Push, SW15 SW_Push, SW16 SW_Push, SW17 SW_Push, SW18 SW_Push, SW19 SW_Push, SW2 SW_Push, SW20 SW_Push, SW21 SW_Push, SW22 SW_Push, SW23 SW_Push, SW24 SW_Push, SW25 SW_Push, SW26 SW_Push, SW27 SW_Push, SW28 SW_Push, SW29 SW_Push, SW3 SW_Push, SW30 SW_Push, SW31 SW_Push, SW32 SW_Push, SW33 SW_Push, SW34 SW_Push, SW35 SW_Push, SW36 SW_Push, SW37 SW_Push, SW38 SW_Push, SW39 SW_Push, SW4 SW_Push, SW40 SW_Push, SW5 SW_Push, SW6 SW_Push, SW7 SW_Push, SW8 SW_Push, SW9 SW_Push, U1 ATmega32U4-M, Y1 16MHz

Commit message: add gerbers
Routing:
- net GND: track 118.5 -> 121.0 mm, vias 7 -> 5
Other:
- board text added: "please work please work please work"
Changed lines of the file:
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@@
     (effects (font (size 1 1) (thickness 0.15)) (justify mirror))
+  )
+  (gr_text "please work please work please work" (at 190.72 17.37) (layer "B.SilkS")
+    (effects (font (size 1.5 1.5) (thickness 0.3)) (justify mirror))
   )
   (segment (start 103.8 32.8755) (end 103.9 32.7755) (width 0.2) (layer "F.Cu") (net 1))
   (segment (start 103.8 34.2245) (end 103.8 32.8755) (width 0.2) (layer "F.Cu") (net 1))
   (segment (start 106.76 24.22) (end 106.888281 24.091719) (width 0.25) (layer "F.Cu") (net 1))
+  (segment (start 106.888281 15.924992) (end 115.528281 15.924992) (width 0.25) (layer "F.Cu") (net 1))
   (segment (start 106.250934 25.669011) (end 106.250934 24.729066) (width 0.25) (layer "F.Cu") (net 1))
   (segment (start 124.666608 29.749986) (end 126.791607 29.749986) (width 0.2) (layer "F.Cu") (net 1))
   (segment (start 106.250934 25.669011) (end 103.9 28.019945) (width 0.25) (layer "F.Cu") (net 1))
-  (segment (start 118.850852 31.935322) (end 118.640466 31.724936) (width 0.25) (layer "F.Cu") (net 1))
   (segment (start 106.888281 24.091719) (end 106.888281 20.104992) (width 0.25) (layer "F.Cu") (net 1))
   (segment (start 106.250934 24.729066) (end 106.76 24.22) (width 0.25) (layer "F.Cu") (net 1))
   (segment (start 115.528281 15.924992) (end 115.528281 20.104992) (width 0.25) (layer "F.Cu") (net 1))
   (segment (start 103.9 28.019945) (end 103.9 32.7755) (width 0.25) (layer "F.Cu") (net 1))
-  (segment (start 118.850852 34.308391) (end 118.850852 31.935322) (width 0.25) (layer "F.Cu") (net 1))
-  (via (at 118.850852 34.308391) (size 0.8) (drill 0.4) (layers "F.Cu" "B.Cu") (net 1))
   (via (at 103.8 34.2245) (size 0.8) (drill 0.4) (layers "F.Cu" "B.Cu") (net 1))
   (via (at 126.791607 29.749986) (size 0.8) (drill 0.4) (layers "F.Cu" "B.Cu") (net 1))
   (via (at 106.76 24.22) (size 0.8) (drill 0.4) (layers "F.Cu" "B.Cu") (net 1))
   (via (at 103.9 32.7755) (size 0.8) (drill 0.4) (layers "F.Cu" "B.Cu") (net 1))
-  (via (at 118.640466 31.724936) (size 0.8) (drill 0.4) (layers "F.Cu" "B.Cu") (net 1))
   (via (at 124.666608 29.749986) (size 0.8) (drill 0.4) (layers "F.Cu" "B.Cu") (net 1))
   (segment (start 110.262526 30.934135) (end 109.617802 30.289411) (width 0.25) (layer "B.Cu") (net 1))
@@
   (segment (start 110.616079 38.836053) (end 110.03 39.422132) (width 0.25) (layer "B.Cu") (net 1))
   (segment (start 111.208281 38.209175) (end 111.208281 34.708317) (width 0.25) (layer "B.Cu") (net 1))
+  (segment (start 116.92151 37.37849) (end 117.422488 37.37849) (width 0.25) (layer "B.Cu") (net 1))
   (segment (start 114.275357 36.361179) (end 112.622495 34.708317) (width 0.25) (layer "B.Cu") (net 1))
   (segment (start 120.6 37.45) (end 120.6 37.85) (width 0.25) (layer "B.Cu") (net 1))
@@
   (segment (start 113.214696 31.994795) (end 111.208281 34.00121) (width 0.25) (layer "B.Cu") (net 1))
   (segment (start 110.03 40.136596) (end 109.791615 40.374981) (width 0.25) (layer "B.Cu") (net 1))
-  (segment (start 117.339411 35.860589) (end 117.739411 35.460589) (width 0.2) (layer "B.Cu") (net 1))
-  (segment (start 118.640466 31.724936) (end 118.640466 31.838356) (width 0.25) (layer "B.Cu") (net 1))
   (segment (start 121.749456 24.739456) (end 118.01 21) (width 0.2) (layer "B.Cu") (net 1))
   (segment (start 110.262526 30.934135) (end 111.208281 31.87989) (width 0.25) (layer "B.Cu") (net 1))
-  (segment (start 118.9 35.65) (end 118.39 35.65) (width 0.25) (layer "B.Cu") (net 1))
+  (segment (start 117.344311 36.955689) (end 116.92151 37.37849) (width 0.25) (layer "B.Cu") (net 1))
   (segment (start 111.208281 34.00121) (end 111.208281 34.708317) (width 0.25) (layer "B.Cu") (net 1))
   (segment (start 119.52 35.03) (end 118.9 35.65) (width 0.25) (layer "B.Cu") (net 1))
@@
   (segment (start 114.275357 36.361179) (end 115.292668 37.37849) (width 0.25) (layer "B.Cu") (net 1))
   (segment (start 130.74 33.82) (end 136.94 33.82) (width 0.2) (layer "B.Cu") (net 1))
-  (segment (start 119.159243 34) (end 118.850852 34.308391) (width 0.25) (layer "B.Cu") (net 1))
   (segment (start 118.9 35.900978) (end 118.9 35.65) (width 0.25) (layer "B.Cu") (net 1))
   (segment (start 119.554322 30.9245) (end 121.7455 30.9245) (width 0.2) (layer "B.Cu") (net 1))
-  (segment (start 118.124011 36.425989) (end 118.9 35.65) (width 0.2) (layer "B.Cu") (net 1))
   (segment (start 120.73 37.98) (end 120.6 37.85) (width 0.25) (layer "B.Cu") (net 1))
   (segment (start 120.73 39.5) (end 120.73 37.98) (width 0.25) (layer "B.Cu") (net 1))
@@
   (segment (start 112.622495 34.708317) (end 111.208281 34.708317) (width 0.25) (layer "B.Cu") (net 1))
   (segment (start 103.9 32.7755) (end 104.795678 32.7755) (width 0.2) (layer "B.Cu") (net 1))
+  (segment (start 117.344311 35.865489) (end 117.344311 36.955689) (width 0.25) (layer "B.Cu") (net 1))
   (segment (start 110.03 39.422132) (end 110.03 40.136596) (width 0.25) (layer "B.Cu") (net 1))
   (segment (start 111.029615 38.422517) (end 111.029615 37.299615) (width 0.25) (layer "B.Cu") (net 1))
   (segment (start 109.085589 30.289411) (end 109.010589 30.214411) (width 0.25) (layer "B.Cu") (net 1))
-  (segment (start 119.52 34) (end 119.159243 34) (width 0.25) (layer "B.Cu") (net 1))
-  (segment (start 117.739411 35.460589) (end 118.710589 35.460589) (width 0.25) (layer "B.Cu") (net 1))
+  (segment (start 115.292668 37.37849) (end 116.92151 37.37849) (width 0.25) (layer "B.Cu") (net 1))
   (segment (start 117.422488 37.37849) (end 118.9 35.900978) (width 0.25) (layer "B.Cu") (net 1))
   (segment (start 118.9 35.65) (end 118.9 35.75) (width 0.25) (layer "B.Cu") (net 1))
@@
   (segment (start 103.74 35) (end 103.74 34.2845) (width 0.2) (layer "B.Cu") (net 1))
   (segment (start 107.75 23.5) (end 107.48 23.5) (width 0.25) (layer "B.Cu") (net 1))
-  (segment (start 115.292668 37.37849) (end 117.422488 37.37849) (width 0.25) (layer "B.Cu") (net 1))
   (segment (start 126.791607 29.749986) (end 126.791607 29.871607) (width 0.2) (layer "B.Cu") (net 1))
+  (segment (start 117.339411 35.860589) (end 117.344311 35.865489) (width 0.25) (layer "B.Cu") (net 1))
   (segment (start 107.434099 33.762562) (end 108.379854 34.708317) (width 0.25) (layer "B.Cu") (net 1))
-  (segment (start 118.640466 31.838356) (end 117.819411 32.659411) (width 0.25) (layer "B.Cu") (net 1))
   (segment (start 110.616079 38.801377) (end 111.208281 38.209175) (width 0.25) (layer "B.Cu") (net 1))
   (segment (start 104.795678 32.7755) (end 105.160589 32.410589) (width 0.2) (layer "B.Cu") (net 1))

Commit message: add minipeg48 and kowgary16
Other:
- board text added: "smol"
- board text removed: "please work please work please work"
Changed lines of the file:
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@@
       (drillshape 0)
       (scaleselection 1)
-      (outputdirectory "gerbers/")
+      (outputdirectory "gerbers-cam350/")
     )
   )
@@
     (effects (font (size 1 1) (thickness 0.15)) (justify mirror))
   )
-  (gr_text "please work please work please work" (at 190.72 17.37) (layer "B.SilkS")
+  (gr_text "smol" (at 190.72 17.37) (layer "B.SilkS")
     (effects (font (size 1.5 1.5) (thickness 0.3)) (justify mirror))
   )
